Commit message: Fixed the absolute path issue for mesh files

File: src/quadro_description/urdf/quadro.ros2_control.xacro (robot description, xacro)
@@ -2,9 +2,107 @@
 <robot xmlns:xacro="http://www.ros.org/wiki/xacro">
   <xacro:macro name="quadro_ros2_control" params="name prefix">
-    <ros2_control name="quadruped_robot" type="system">
+<ros2_control name="quadruped_robot" type="system">
     <hardware>
         <plugin>gz_ros2_control/GazeboSimSystem</plugin>
     </hardware>
-    <joint name="Base-Body_Revolute-41">
+    <joint name="rear_right_joint_1">
+        <command_interface name="position">
+            <!-- <param name="min">-0.349066</param> -->
+            <!-- <param name="max">0.349066</param> -->
+            <initial_value>0.062832</initial_value>
+        </command_interface>
+        <state_interface name="position"/>
+        <state_interface name="velocity"/>
+        <state_interface name="effort"/>
+    </joint>
+    <joint name="rear_right_joint_2">
+        <command_interface name="position">
+            <!-- <param name="min">-0.349066</param> -->
+            <!-- <param name="max">0.349066</param> -->
+        </command_interface>
+        <state_interface name="position">
+            <initial_value>-0.753982</initial_value>
+        </state_interface>
+        <state_interface name="velocity"/>
+        <state_interface name="effort"/>
+    </joint>
+    <joint name="rear_right_joint_3">
+        <command_interface name="position">
+            <!-- <param name="min">-0.349066</param> -->
+            <!-- <param name="max">0.349066</param> -->
+        </command_interface>
+        <state_interface name="position">
+            <initial_value>0.753982</initial_value>
+        </state_interface>
+        <state_interface name="velocity"/>
+        <state_interface name="effort"/>
+        <!-- <param name="min">-0.349066</param> -->
+        <!-- <param name="max">0.349066</param> -->
+    </joint>
+    <joint name="rear_left_joint_1">
+        <command_interface name="position">
+            <!-- <param name="min">-0.349066</param> -->
+            <!-- <param name="max">0.349066</param> -->
+        </command_interface>
+        <state_interface name="position">
+            <initial_value>-0.125664</initial_value>
+        </state_interface>
+        <state_interface name="velocity"/>
+        <state_interface name="effort"/>
+    </joint>
+    <joint name="rear_left_joint_2">
+        <command_interface name="position">
+            <!-- <param name="min">-0.349066</param> -->
+            <!-- <param name="max">0.349066</param> -->
+        </command_interface>
+        <state_interface name="position">
+            <initial_value>0.565487</initial_value>
+        </state_interface>
+        <state_interface name="velocity"/>
+        <state_interface name="effort"/>
+    </joint>
+    <joint name="rear_left_joint_3">
+        <command_interface name="position">
+            <!-- <param name="min">-0.349066</param> -->
+            <!-- <param name="max">0.349066</param> -->
+        </command_interface>
+        <state_interface name="position">
+            <initial_value>-1.193805</initial_value>
+        </state_interface>
+        <state_interface name="velocity"/>
+        <state_interface name="effort"/>
+    </joint>
+    <joint name="front_right_joint_1">
+        <command_interface name="position">
+            <!-- <param name="min">-0.349066</param> -->
+            <!-- <param name="max">0.349066</param> -->
+        </command_interface>
+        <state_interface name="position">
+            <initial_value>-0.125664</initial_value>
+        </state_interface>
+        <state_interface name="velocity"/>
+        <state_interface name="effort"/>
+        <!-- <param name="min">-0.349066</param> -->
+        <!-- <param name="max">0.349066</param> -->
+    </joint>
+    <joint name="front_right_joint_2">
+        <command_interface name="position">
+            <!-- <param name="min"/>-0.349066</param> -->
+            <!-- <param name="max"/>0.349066</param> -->
+        </command_interface>
+        <state_interface name="position"/>
+        <state_interface name="velocity"/>
+        <state_interface name="effort"/>
+    </joint>
+    <joint name="front_right_joint_3">
+        <command_interface name="position">
+            <!-- <param name="min">-0/.349066</param> -->
+            <!-- <param name="max">0./349066</param> -->
+        </command_interface>
+        <state_interface name="position"/>
+        <state_interface name="velocity"/>
+        <state_interface name="effort"/>
+    </joint>
+    <joint name="front_left_joint_1">
         <command_interface name="position">
             <!-- <param name="min">-0.349066</param> -->
@@ -15,5 +113,5 @@
         <state_interface name="effort"/>
     </joint>
-    <joint name="Actuator-1_Revolute-61">
+    <joint name="front_left_joint_2">
         <command_interface name="position">
             <!-- <param name="min">-0.349066</param> -->
@@ -24,92 +122,5 @@
         <state_interface name="effort"/>
     </joint>
-    <joint name="Base-Body_Revolute-62">
-        <command_interface name="position">
-            <!-- <param name="min">-0.349066</param> -->
-            <!-- <param name="max">0.349066</param> -->
-        </command_interface>
-        <state_interface name="position"/>
-        <state_interface name="velocity"/>
-        <state_interface name="effort"/>
-        <!-- <param name="min">-0.349066</param> -->
-        <!-- <param name="max">0.349066</param> -->
-    </joint>
-    <joint name="Actuator-2_Revolute-63">
-        <command_interface name="position">
-            <!-- <param name="min">-0.349066</param> -->
-            <!-- <param name="max">0.349066</param> -->
-        </command_interface>
-        <state_interface name="position"/>
-        <state_interface name="velocity"/>
-        <state_interface name="effort"/>
-    </joint>
-    <joint name="Base-Body_Revolute-64">
-        <command_interface name="position">
-            <!-- <param name="min">-0.349066</param> -->
-            <!-- <param name="max">0.349066</param> -->
-        </command_interface>
-        <state_interface name="position"/>
-        <state_interface name="velocity"/>
-        <state_interface name="effort"/>
-        <!-- <param name="min">-0.349066</param> -->
-        <!-- <param name="max">0.349066</param> -->
-    </joint>
-    <joint name="Actuator-3_Revolute-65">
-        <command_interface name="position">
-            <!-- <param name="min">-0.349066</param> -->
-            <!-- <param name="max">0.349066</param> -->
-        </command_interface>
-        <state_interface name="position"/>
-        <state_interface name="velocity"/>
-        <state_interface name="effort"/>
-    </joint>
-    <joint name="Base-Body_Revolute-66">
-        <command_interface name="position">
-            <!-- <param name="min">-0.349066</param> -->
-            <!-- <param name="max">0.349066</param> -->
-        </command_interface>
-        <state_interface name="position"/>
-        <state_interface name="velocity"/>
-        <state_interface name="effort"/>
-        <!-- <param name="min">-0.349066</param> -->
-        <!-- <param name="max">0.349066</param> -->
-    </joint>
-    <joint name="Actuator-4_Revolute-67">
-        <command_interface name="position">
-            <!-- <param name="min"/>-0.349066</param> -->
-            <!-- <param name="max"/>0.349066</param> -->
-        </command_interface>
-        <state_interface name="position"/>
-        <state_interface name="velocity"/>
-        <state_interface name="effort"/>
-    </joint>
-    <joint name="upper-leg-1_Revolute-68">
-        <command_interface name="position">
-            <!-- <param name="min">-0/.349066</param> -->
-            <!-- <param name="max">0./349066</param> -->
-        </command_interface>
-        <state_interface name="position"/>
-        <state_interface name="velocity"/>
-        <state_interface name="effort"/>
-    </joint>
-    <joint name="upper-leg-2_Revolute-69">
-        <command_interface name="position">
-            <!-- <param name="min">-0.349066</param> -->
-            <!-- <param name="max">0.349066</param> -->
-        </command_interface>
-        <state_interface name="position"/>
-        <state_interface name="velocity"/>
-        <state_interface name="effort"/>
-    </joint>
-    <joint name="upper-leg-3_Revolute-70">
-        <command_interface name="position">
-            <!-- <param name="min">-0.349066</param> -->
-            <!-- <param name="max">0.349066</param> -->
-        </command_interface>
-        <state_interface name="position"/>
-        <state_interface name="velocity"/>
-        <state_interface name="effort"/>
-    </joint>
-    <joint name="upper-leg-4_Revolute-71">
+    <joint name="front_left_joint_3">
         <command_interface name="position">
             <!-- <param name="min">-0.349066</param> -->
