Commit message: Xacro preparation successfull

File: src/quadro_description/urdf/quadro_description.urdf.xacro (robot description, xacro)
@@ -1,4 +1,7 @@
-<?xml version='1.0' encoding='utf-8'?>
-<robot name="Demo">
+<?xml version="1.0"?>
+<robot xmlns:xacro="http://www.ros.org/wiki/xacro">
+  <xacro:macro name="quadro" params="parent prefix *origin">
+  <!-- Constants for robot dimensions -->
+  <!-- Base Link -->
  <link name="Base-Body">
         <inertial>
@@ -363,3 +366,4 @@
         <axis xyz="1.3877787807814457e-17 -1.0 1.894318035766673e-15" />
     </joint>
+  </xacro:macro>
 </robot>

Commit message: changed mesh file path

File: src/quadro_description/urdf/quadro_description.urdf.xacro (robot description, xacro)
@@ -1,385 +1,497 @@
 <?xml version="1.0"?>
 <robot xmlns:xacro="http://www.ros.org/wiki/xacro">
-  <xacro:macro name="quadro" params="parent prefix *origin">
-  <!-- Constants for robot dimensions -->
-  <!-- Base Link -->
-  <link name="base_link">
-</link>
- <link name="base_body">
-        <inertial>
-            <origin xyz="-7.493020562650216e-16 -4.84842506995014e-16 0.05771131130384984" rpy="0.0 0.0 0.0" />
-            <mass value="1.91682581128143" />
-            <inertia ixx="0.7997201982029933" iyy="1.206821240279861" izz="1.846293564893905" ixy="-6.5797939896583456e-15" iyz="-8.547383638323425e-17" ixz="5.242219058711254e-16" />
-        </inertial>
-        <visual name="base_body_visual">
+    <xacro:macro name="quadro" params="parent prefix *origin">
+        <!-- Constants for robot dimensions -->
+        <!-- Base Link -->
+        <link name="base_link">
+        </link>
+        <link name="base_body">
+            <inertial>
+                <origin xyz="-7.493020562650216e-16 -4.84842506995014e-16 0.05771131130384984"
+                    rpy="0.0 0.0 0.0" />
+                <mass value="1.91682581128143" />
+                <inertia ixx="0.7997201982029933" iyy="1.206821240279861" izz="1.846293564893905"
+                    ixy="-6.5797939896583456e-15" iyz="-8.547383638323425e-17"
+                    ixz="5.242219058711254e-16" />
+            </inertial>
+            <visual name="base_body_visual">
+                <origin xyz="0.0 0.0 0.0" rpy="0.0 0.0 0.0" />
+                <geometry>
+                    <mesh
+                        filename="/home/jarin/quadro_robot/src/quadro_description/urdf/meshes/base_body.stl"
+                        scale="0.001 0.001 0.001" />
+                </geometry>
+                <material name="yellow">
+                    <color rgba="0.8 0.8 0.0 1.0" />
+                </material>
+            </visual>
+            <collision name="base_body_collision">
+                <origin xyz="0.0 0.0 0.0" rpy="0.0 0.0 0.0" />
+                <geometry>
+                    <mesh
+                        filename="/home/jarin/quadro_robot/src/quadro_description/urdf/meshes/base_body.stl"
+                        scale="0.001 0.001 0.001" />
+                </geometry>
+            </collision>
+        </link>
+        <link name="actuator_rear_right">
+            <inertial>
+                <origin xyz="-3.9968028886505636e-16 -1.7763568394002506e-16 0.07768426014187582"
+                    rpy="0.0 -0.0 0.0" />
+                <mass value="1.077991723221682" />
+                <inertia ixx="0.09357165466628592" iyy="0.10577974343263863"
+                    izz="0.054310757474580806" ixy="5.551115123125783e-17"
+                    iyz="2.220446049250313e-15" ixz="0.0" />
+            </inertial>
+            <visual name="actuator_rear_right_visual">
+                <origin xyz="-4.263256414560601e-16 -3.1974423109204507e-16 0.23999999999999994"
+                    rpy="3.1415926535897887 5.3672300325485344e-17 3.141592653589793" />
+                <geometry>
+                    <mesh
+                        filename="/home/jarin/quadro_robot/src/quadro_description/urdf/meshes/actuator_rear_right.stl"
+                        scale="0.001 0.001 0.001" />
+                </geometry>
+                <material name="black">
+                    <color rgba="0.0 0.0 0.0 1.0" />
+                </material>
+            </visual>
+            <collision name="actuator_rear_right_collision">
+                <origin xyz="-4.263256414560601e-16 -3.1974423109204507e-16 0.23999999999999994"
+                    rpy="3.1415926535897887 5.3672300325485344e-17 3.141592653589793" />
+                <geometry>
+                    <mesh
+                        filename="/home/jarin/quadro_robot/src/quadro_description/urdf/meshes/actuator_rear_right.stl"
+                        scale="0.001 0.001 0.001" />
+                </geometry>
+            </collision>
+        </link>
+        <link name="actuator_rear_left">
+            <inertial>
+                <origin xyz="5.329070518200751e-17 -3.552713678800501e-17 0.07768426014187589"
+                    rpy="0.0 -0.0 0.0" />
+                <mass value="1.077991723221682" />
+                <inertia ixx="0.09357165466628592" iyy="0.10577974343263774"
+                    izz="0.05431075747458092" ixy="5.551115123125783e-17"
+                    iyz="2.220446049250313e-15" ixz="1.1102230246251565e-16" />
+            </inertial>
+            <visual name="actuator_rear_left_visual">
+                <origin xyz="3.552713678800501e-17 -1.7763568394002506e-16 0.24"
+                    rpy="3.1415926535897887 5.36723003254851e-17 3.141592653589793" />
+                <geometry>
+                    <mesh
+                        filename="/home/jarin/quadro_robot/src/quadro_description/urdf/meshes/actuator_rear_left.stl"
+                        scale="0.001 0.001 0.001" />
+                </geometry>
+                <material name="black">
+                    <color rgba="0.0 0.0 0.0 1.0" />
+                </material>
+            </visual>
+            <collision name="actuator_rear_left_collision">
+                <origin xyz="3.552713678800501e-17 -1.7763568394002506e-16 0.24"
+                    rpy="3.1415926535897887 5.36723003254851e-17 3.141592653589793" />
+                <geometry>
+                    <mesh
+                        filename="/home/jarin/quadro_robot/src/quadro_description/urdf/meshes/actuator_rear_left.stl"
+                        scale="0.001 0.001 0.001" />
+                </geometry>
+            </collision>
+        </link>
+        <link name="actuator_front_right">
+            <inertial>
+                <origin xyz="-1.7763568394002505e-17 7.105427357601002e-17 0.07768426014187568"
+                    rpy="0.0 -0.0 0.0" />
+                <mass value="1.077991723221682" />
+                <inertia ixx="0.09357165466629214" iyy="0.1057797434326413"
+                    izz="0.054310757474580806" ixy="0.0" iyz="0.0" ixz="1.1102230246251565e-16" />
+            </inertial>
+            <visual name="actuator_front_right_visual">
+                <origin xyz="0.0 7.105427357601002e-17 0.23999999999999985"
+                    rpy="3.141592653589793 -0.0 0.0" />
+                <geometry>
+                    <mesh
+                        filename="/home/jarin/quadro_robot/src/quadro_description/urdf/meshes/actuator_front_right.stl"
+                        scale="0.001 0.001 0.001" />
+                </geometry>
+                <material name="black">
+                    <color rgba="0.0 0.0 0.0 1.0" />
+                </material>
+            </visual>
+            <collision name="actuator_front_right_collision">
+                <origin xyz="0.0 7.105427357601002e-17 0.23999999999999985"
+                    rpy="3.141592653589793 -0.0 0.0" />
+                <geometry>
+                    <mesh
+                        filename="/home/jarin/quadro_robot/src/quadro_description/urdf/meshes/actuator_front_right.stl"
+                        scale="0.001 0.001 0.001" />
+                </geometry>
+            </collision>
+        </link>
+        <link name="actuator_front_left">
+            <inertial>
+                <origin xyz="-1.7763568394002505e-17 -7.105427357601002e-17 0.07768426014187568"
+                    rpy="0.0 -0.0 0.0" />
+                <mass value="1.077991723221682" />
+                <inertia ixx="0.09357165466629214" iyy="0.1057797434326413"
+                    izz="0.054310757474580806" ixy="-5.551115123125783e-17" iyz="0.0"
+                    ixz="1.1102230246251565e-16" />
+            </inertial>
+            <visual name="actuator_front_left_visual">
+                <origin xyz="0.0 -7.105427357601002e-17 0.23999999999999985"
+                    rpy="3.141592653589793 -0.0 0.0" />
+                <geometry>
+                    <mesh
+                        filename="/home/jarin/quadro_robot/src/quadro_description/urdf/meshes/actuator_front_left.stl"
+                        scale="0.001 0.001 0.001" />
+                </geometry>
+                <material name="black">
+                    <color rgba="0.0 0.0 0.0 1.0" />
+                </material>
+            </visual>
+            <collision name="actuator_front_left_collision">
+                <origin xyz="0.0 -7.105427357601002e-17 0.23999999999999985"
+                    rpy="3.141592653589793 -0.0 0.0" />
+                <geometry>
+                    <mesh
+                        filename="/home/jarin/quadro_robot/src/quadro_description/urdf/meshes/actuator_front_left.stl"
+                        scale="0.001 0.001 0.001" />
+                </geometry>
+            </collision>
+        </link>
+        <link name="upper-leg-1">
+            <inertial>
+                <origin xyz="-0.0349227234083768 0.020547382026482666 -0.04559883324274818"
+                    rpy="-2.189528850507527e-47 1.2154326714572545e-63 6.842277657836022e-49" />
+                <mass value="1.100857588170285" />
+                <inertia ixx="0.06465148006887686" iyy="0.12169393436924025"
+                    izz="0.1633221816047396" ixy="0.05133169967548328" iyz="0.01087298230174924"
+                    ixz="-0.018479928638119193" />
+            </inertial>
+            <visual name="upper-leg-1_visual">
+                <origin xyz="-0.8515680735795619 0.5095601952053456 -0.30000000000000165"
+                    rpy="-4.225104217839752e-15 1.3947237586551614e-15 1.5707963267948966" />
+                <geometry>
+                    <mesh
+                        filename="/home/jarin/quadro_robot/src/quadro_description/urdf/meshes/upper-leg-1.stl"
+                        scale="0.001 0.001 0.001" />
+                </geometry>
+                <material name="yellow">
+                    <color rgba="1.0 1.0 0.0 1.0" />
+                </material>
+            </visual>
+            <collision name="upper-leg-1_collision">
+                <origin xyz="-0.8515680735795619 0.5095601952053456 -0.30000000000000165"
+                    rpy="-4.225104217839752e-15 1.3947237586551614e-15 1.5707963267948966" />
+                <geometry>
+                    <mesh
+                        filename="/home/jarin/quadro_robot/src/quadro_description/urdf/meshes/upper-leg-1.stl"
+                        scale="0.001 0.001 0.001" />
+                </geometry>
+            </collision>
+        </link>
+        <link name="upper-leg-2">
+            <inertial>
+                <origin xyz="-0.0352559165208968 -0.019970274628070613 -0.04559883324293296"
+                    rpy="0.0 -1.2154326714572545e-63 -6.842277657836022e-49" />
+                <mass value="1.100857588155373" />
+                <inertia ixx="0.06297876485799389" iyy="0.1233666495886574" izz="0.163322181612584"
+                    ixy="-0.05036595710029217" iyz="-0.010567596510820206"
+                    ixz="-0.018656243209292257" />
+            </inertial>
+            <visual name="upper-leg-2_visual">
+                <origin xyz="-0.517058214677661 0.2407886725118906 0.7308212118024103"
+                    rpy="-3.141592653589791 -6.2920377852306045e-15 2.617993877991495" />
+                <geometry>
+                    <mesh
+                        filename="/home/jarin/quadro_robot/src/quadro_description/urdf/meshes/upper-leg-2.stl"
+                        scale="0.001 0.001 0.001" />
+                </geometry>
+                <material name="yellow">
+                    <color rgba="1.0 1.0 0.0 1.0" />
+                </material>
+            </visual>
+            <collision name="upper-leg-2_collision">
+                <origin xyz="-0.517058214677661 0.2407886725118906 0.7308212118024103"
+                    rpy="-3.141592653589791 -6.2920377852306045e-15 2.617993877991495" />
+                <geometry>
+                    <mesh
+                        filename="/home/jarin/quadro_robot/src/quadro_description/urdf/meshes/upper-leg-2.stl"
+                        scale="0.001 0.001 0.001" />
+                </geometry>
+            </collision>
+        </link>
+        <link name="upper-leg-3">
+            <inertial>
+                <origin xyz="0.020547382026482097 0.03492272340837815 -0.045598833242747966"
+                    rpy="0.0 -0.0 0.0" />
+                <mass value="1.100857588170285" />
+                <inertia ixx="0.12169393436921117" iyy="0.0646514800688931"
+                    izz="0.16332218160470413" ixy="-0.05133169967548612" iyz="0.018479928638120383"
+                    ixz="0.010872982301734394" />
+            </inertial>
+            <visual name="upper-leg-3_visual">
+                <origin xyz="0.5095601952053488 0.8515680735795635 -0.2999999999999954"
+                    rpy="4.67577335227251e-16 -2.6941296856217734e-15 -3.683442676833609e-15" />
+                <geometry>
+                    <mesh
+                        filename="/home/jarin/quadro_robot/src/quadro_description/urdf/meshes/upper-leg-3.stl"
+                        scale="0.001 0.001 0.001" />
+                </geometry>
+                <material name="yellow">
+                    <color rgba="1.0 1.0 0.0 1.0" />
+                </material>
+            </visual>
+            <collision name="upper-leg-3_collision">
+                <origin xyz="0.5095601952053488 0.8515680735795635 -0.2999999999999954"
+                    rpy="4.67577335227251e-16 -2.6941296856217734e-15 -3.683442676833609e-15" />
+                <geometry>
+                    <mesh
+                        filename="/home/jarin/quadro_robot/src/quadro_description/urdf/meshes/upper-leg-3.stl"
+                        scale="0.001 0.001 0.001" />
+                </geometry>
+            </collision>
+        </link>
+        <link name="upper-leg-4">
+            <inertial>
+                <origin xyz="-0.01742547713701903 -0.03658065424438789 -0.045598833242747966"
+                    rpy="0.0 -0.0 0.0" />
+                <mass value="1.100857588170285" />
+                <inertia ixx="0.1301742889471318" iyy="0.05617112549094383" izz="0.1633221816048973"
+                    ixy="-0.045599196696266164" iyz="-0.019357249778792916"
+                    ixz="-0.009220975415064496" />
+            </inertial>
+            <visual name="upper-leg-4_visual">
+                <origin xyz="-0.43340211686914304 -0.8927386972519166 -0.29999999999999816"
+                    rpy="-1.9956054263512081e-16 2.024318169035165e-15 -3.0543261909900847" />
+                <geometry>
+                    <mesh
+                        filename="/home/jarin/quadro_robot/src/quadro_description/urdf/meshes/upper-leg-4.stl"
+                        scale="0.001 0.001 0.001" />
+                </geometry>
+                <material name="yellow">
+                    <color rgba="1.0 1.0 0.0 1.0" />
+                </material>
+            </visual>
+            <collision name="upper-leg-4_collision">
+                <origin xyz="-0.43340211686914304 -0.8927386972519166 -0.29999999999999816"
+                    rpy="-1.9956054263512081e-16 2.024318169035165e-15 -3.0543261909900847" />
+                <geometry>
+                    <mesh
+                        filename="/home/jarin/quadro_robot/src/quadro_description/urdf/meshes/upper-leg-4.stl"
+                        scale="0.001 0.001 0.001" />
+                </geometry>
+            </collision>
+        </link>
+        <link name="lower-leg-1">
+            <inertial>
+                <origin xyz="-0.10712098868393852 -0.00689898677812046 0.08067764538747335"
+                    rpy="0.0 -0.0 0.0" />
+                <mass value="1.9006674864295967" />
+                <inertia ixx="0.009619790261939432" iyy="0.02503802990092563"
+                    izz="0.015603429466196646" ixy="-3.195877794574224e-05"
+                    iyz="2.4069596516153475e-05" ixz="0.010413204731261842" />
+            </inertial>
+            <visual name="lower-leg-1_visual">
+                <origin xyz="-0.5499084735795644 0.18000000000000033 0.33207360520534585"
+                    rpy="1.5707963267948943 -1.5707963267948957 0" />
+                <geometry>
+                    <mesh filename="$(find quadro_description)/urdf/meshes/lower-leg-1.stl"
+                        scale="0.001 0.001 0.001" />
+                </geometry>
+                <material name="black">
+                    <color rgba="0.0 0.0 0.0 1.0" />
+                </material>
+            </visual>
+            <collision name="lower-leg-1_collision">
+                <origin xyz="-0.5499084735795644 0.18000000000000033 0.33207360520534585"
+                    rpy="1.5707963267948943 -1.5707963267948957 0" />
+                <geometry>
+                    <mesh filename="$(find quadro_description)/urdf/meshes/lower-leg-1.stl"
+                        scale="0.001 0.001 0.001" />
+                </geometry>
+            </collision>
+        </link>
+        <link name="lower-leg-2">
+            <inertial>
+                <origin xyz="-0.12342939053611061 -0.006898986778124297 -0.052430676680511094"
+                    rpy="0.0 -0.0 0.0" />
+                <mass value="1.9006674864295967" />
+                <inertia ixx="0.005089419833048475" iyy="0.025038029900930736"
+                    izz="0.020133799895080157" ixy="-3.6824271014769076e-05"
+                    iyz="-1.5642315316679312e-05" ixz="-0.007797594144611351" />
+            </inertial>
+            <visual name="lower-leg-2_visual">
+                <origin xyz="-0.5625384205949758 0.17999999999999347 -0.3101979071690065"
+                    rpy="-1.5707963267948921 -0.5235987755982989 -3.1415926535897913" />
+                <geometry>
+                    <mesh filename="$(find quadro_description)/urdf/meshes/lower-leg-2.stl"
+                        scale="0.001 0.001 0.001" />
+                </geometry>
+                <material name="black">
+                    <color rgba="0.0 0.0 0.0 1.0" />
+                </material>
+            </visual>
+            <collision name="lower-leg-2_collision">
+                <origin xyz="-0.5625384205949758 0.17999999999999347 -0.3101979071690065"
+                    rpy="-1.5707963267948921 -0.5235987755982989 -3.1415926535897913" />
+                <geometry>
+                    <mesh filename="$(find quadro_description)/urdf/meshes/lower-leg-2.stl"
+                        scale="0.001 0.001 0.001" />
+                </geometry>
+            </collision>
+        </link>
+        <link name="lower-leg-3">
+            <inertial>
+                <origin xyz="0.08067764538747434 -0.006898986778123409 0.10712098868393938"
+                    rpy="0.0 -0.0 0.0" />
+                <mass value="1.9006674864295967" />
+                <inertia ixx="0.015603429466191032" iyy="0.02503802990093118"
+                    izz="0.009619790261938148" ixy="2.406959651638755e-05"
+                    iyz="3.1958777945982564e-05" ixz="-0.010413204731259892" />
+            </inertial>
+            <visual name="lower-leg-3_visual">
+                <origin xyz="0.33207360520535056 0.17999999999999594 0.5499084735795655"
+                    rpy="1.5707963267948968 3.683442676833602e-15 -5.4696434248321024e-15" />
+                <geometry>
+                    <mesh filename="$(find quadro_description)/urdf/meshes/lower-leg-3.stl"
+                        scale="0.001 0.001 0.001" />
+                </geometry>
+                <material name="black">
+                    <color rgba="0.0 0.0 0.0 1.0" />
+                </material>
+            </visual>
+            <collision name="lower-leg-3_collision">
+                <origin xyz="0.33207360520535056 0.17999999999999594 0.5499084735795655"
+                    rpy="1.5707963267948968 3.683442676833602e-15 -5.4696434248321024e-15" />
+                <geometry>
+                    <mesh filename="$(find quadro_description)/urdf/meshes/lower-leg-3.stl"
+                        scale="0.001 0.001 0.001" />
+                </geometry>
+            </collision>
+        </link>
+        <link name="lower-leg-4">
+            <inertial>
+                <origin xyz="-0.07103443670234136 0.006898986778121526 0.11374488081583926"
+                    rpy="0.0 -0.0 -9.339709002946167e-47" />
+                <mass value="1.9006674864295967" />
+                <inertia ixx="0.017366211029108014" iyy="0.025038029900934677"
+                    izz="0.007857008699020403" ixy="2.119261340548661e-05"
+                    iyz="-3.39349687089089e-05" ixz="0.009735480731230683" />
+            </inertial>
+            <visual name="lower-leg-4_visual">
+                <origin xyz="-0.28288228686915 -0.17999999999999727 0.5767580272519269"
+                    rpy="1.5707963267949006 -0.08726646259970866 3.1415926535897927" />
+                <geometry>
+                    <mesh filename="$(find quadro_description)/urdf/meshes/lower-leg-4.stl"
+                        scale="0.001 0.001 0.001" />
+                </geometry>
+                <material name="black">
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